Commit message: fixes

File: urdf/saminda_bot.xacro (robot description, xacro)
@@ -23,7 +23,7 @@
             <origin xyz="0.0 0 0" rpy=" 0 0 0"/>
             <inertia
-                    ixx="0.147116667" ixy="0" ixz="0"
-                    iyy="0.334951167" iyz="0"
-                    izz="0.3978345"
+                    ixx="0.1" ixy="0" ixz="0"
+                    iyy="0.1" iyz="0"
+                    izz="0.1"
             />
         </inertial>
@@ -31,5 +31,5 @@
             <origin xyz="0 0 0" rpy=" 0 0 0"/>
             <geometry>
-                <box size="0.5 0.3 0.05"/>
+                <box size="0.4 0.2 0.05"/>
             </geometry>
         </collision>
@@ -37,5 +37,5 @@
             <origin xyz="0 0 0" rpy=" 0 0 0"/>
             <geometry>
-                <box size="0.5 0.3 0.05"/>
+                <box size="0.4 0.2 0.05"/>
             </geometry>
             <material name="blue"/>
@@ -43,22 +43,21 @@
     </link>
     <link name='right_front_wheel'>
-        <pose>0.25 -0.18 0 1.5707 0 0</pose>
-        <inertial>
-            <mass value="0.2"/>
-            <!-- <origin xyz="0.0 0 0" rpy="0 1.5707 1.5707"/> -->
-            <inertia
-                    ixx="0.005240625" ixy="0" ixz="0"
-                    iyy="0.005240625" iyz="0"
-                    izz="0.009075"
-            />
-        </inertial>
-        <collision name='collision'>
-            <!-- <origin xyz="0 0 0" rpy="0 1.5707 1.5707"/>  -->
-            <geometry>
-                <cylinder length="0.0375" radius="0.055"/>
-            </geometry>
-        </collision>
-        <visual name='visual'>
-            <!-- <origin xyz="0 0 0" rpy="0 1.5707 1.5707"/> -->
+        <inertial>
+            <mass value="0.2"/>
+             <origin xyz="0.0 0 0" rpy="1.5707 0 0"/>
+            <inertia
+                    ixx="0.005" ixy="0" ixz="0"
+                    iyy="0.005" iyz="0"
+                    izz="0.005"
+            />
+        </inertial>
+        <collision name='collision'>
+             <origin xyz="0 0 0" rpy="1.5707 0 0"/>
+            <geometry>
+                <cylinder length="0.0375" radius="0.055"/>
+            </geometry>
+        </collision>
+        <visual name='visual'>
+             <origin xyz="0 0 0" rpy="1.5707 0 0"/>
             <geometry>
                 <cylinder length="0.0375" radius="0.055"/>
@@ -68,22 +67,21 @@
     </link>
     <link name='left_front_wheel'>
-        <pose>0.25 0.18 0 1.5707 0 0</pose>
-        <inertial>
-            <mass value="0.2"/>
-            <!-- <origin xyz="0.0 0 0" rpy="0 1.5707 1.5707"/> -->
-            <inertia
-                    ixx="0.005240625" ixy="0" ixz="0"
-                    iyy="0.005240625" iyz="0"
-                    izz="0.009075"
-            />
-        </inertial>
-        <collision name='collision'>
-            <!-- <origin xyz="0 0 0" rpy="0 1.5707 1.5707"/>  -->
-            <geometry>
-                <cylinder length="0.0375" radius="0.055"/>
-            </geometry>
-        </collision>
-        <visual name='visual'>
-            <!-- <origin xyz="0 0 0" rpy="0 1.5707 1.5707"/> -->
+        <inertial>
+            <mass value="0.2"/>
+             <origin xyz="0.0 0 0" rpy="1.5707 0 0"/>
+            <inertia
+                    ixx="0.005" ixy="0" ixz="0"
+                    iyy="0.005" iyz="0"
+                    izz="0.005"
+            />
+        </inertial>
+        <collision name='collision'>
+             <origin xyz="0 0 0" rpy="1.5707 0 0"/>
+            <geometry>
+                <cylinder length="0.0375" radius="0.055"/>
+            </geometry>
+        </collision>
+        <visual name='visual'>
+             <origin xyz="0 0 0" rpy="1.5707 0 0"/>
             <geometry>
                 <cylinder length="0.0375" radius="0.055"/>
@@ -93,22 +91,21 @@
     </link>
     <link name='right_rear_wheel'>
-        <pose>-0.25 -0.18 0 1.5707 0 0</pose>
-        <inertial>
-            <mass value="0.2"/>
-            <!-- <origin xyz="0.0 0 0" rpy="0 1.5707 1.5707"/> -->
-            <inertia
-                    ixx="0.005240625" ixy="0" ixz="0"
-                    iyy="0.005240625" iyz="0"
-                    izz="0.009075"
-            />
-        </inertial>
-        <collision name='collision'>
-            <!-- <origin xyz="0 0 0" rpy="0 1.5707 1.5707"/>  -->
-            <geometry>
-                <cylinder length="0.0375" radius="0.055"/>
-            </geometry>
-        </collision>
-        <visual name='visual'>
-            <!-- <origin xyz="0 0 0" rpy="0 1.5707 1.5707"/> -->
+        <inertial>
+            <mass value="0.2"/>
+             <origin xyz="0.0 0 0" rpy="1.5707 0 0"/>
+            <inertia
+                    ixx="0.005" ixy="0" ixz="0"
+                    iyy="0.005" iyz="0"
+                    izz="0.005"
+            />
+        </inertial>
+        <collision name='collision'>
+             <origin xyz="0 0 0" rpy="1.5707 0 0"/>
+            <geometry>
+                <cylinder length="0.0375" radius="0.055"/>
+            </geometry>
+        </collision>
+        <visual name='visual'>
+             <origin xyz="0 0 0" rpy="1.5707 0 0"/>
             <geometry>
                 <cylinder length="0.0375" radius="0.055"/>
@@ -118,22 +115,21 @@
     </link>
     <link name='left_rear_wheel'>
-        <pose>-0.25 0.18 0 1.5707 0 0</pose>
-        <inertial>
-            <mass value="0.2"/>
-            <!-- <origin xyz="0.0 0 0" rpy="0 1.5707 1.5707"/> -->
-            <inertia
-                    ixx="0.005240625" ixy="0" ixz="0"
-                    iyy="0.005240625" iyz="0"
-                    izz="0.009075"
-            />
-        </inertial>
-        <collision name='collision'>
-            <!-- <origin xyz="0 0 0" rpy="0 1.5707 1.5707"/>  -->
-            <geometry>
-                <cylinder length="0.0375" radius="0.055"/>
-            </geometry>
-        </collision>
-        <visual name='visual'>
-            <!-- <origin xyz="0 0 0" rpy="0 1.5707 1.5707"/> -->
+        <inertial>
+            <mass value="0.2"/>
+             <origin xyz="0.0 0 0" rpy="1.5707 0 0"/>
+            <inertia
+                    ixx="0.005" ixy="0" ixz="0"
+                    iyy="0.005" iyz="0"
+                    izz="0.005"
+            />
+        </inertial>
+        <collision name='collision'>
+             <origin xyz="0 0 0" rpy="1.5707 0 0"/>
+            <geometry>
+                <cylinder length="0.0375" radius="0.055"/>
+            </geometry>
+        </collision>
+        <visual name='visual'>
+             <origin xyz="0 0 0" rpy="1.5707 0 0"/>
             <geometry>
                 <cylinder length="0.0375" radius="0.055"/>
@@ -189,6 +185,6 @@
         </visual>
     </link>
-    <joint type="revolute" name="right_front">
-        <pose>0 0 0 0 0 0</pose>
+    <joint type="continuous" name="right_front">
+        <origin xyz="0.15 -0.13 0" rpy="0 0 0"/>
         <child link="right_front_wheel"/>
         <parent link="chassis"/>
@@ -197,6 +193,6 @@
         <dynamics damping="1.0" friction="1.0"/>
     </joint>
-    <joint type="revolute" name="right_rear">
-        <pose>0 0 0 0 0 0</pose>
+    <joint type="continuous" name="right_rear">
+        <origin xyz="-0.15 -0.13 0" rpy="0 0 0"/>
         <child link="right_rear_wheel"/>
         <parent link="chassis"/>
@@ -205,6 +201,6 @@
         <dynamics damping="1.0" friction="1.0"/>
     </joint>
-    <joint type="revolute" name="left_front">
-        <pose>0 0 0 0 0 0</pose>
+    <joint type="continuous" name="left_front">
+        <origin xyz="0.15 0.13 0" rpy="0 0 0"/>
         <child link="left_front_wheel"/>
         <parent link="chassis"/>
@@ -213,6 +209,6 @@
         <dynamics damping="1.0" friction="1.0"/>
     </joint>
-    <joint type="revolute" name="left_rear">
-        <pose>0 0 0 0 0 0</pose>
+    <joint type="continuous" name="left_rear">
+        <origin xyz="-0.15 0.13 0" rpy="0 0 0"/>
         <child link="left_rear_wheel"/>
         <parent link="chassis"/>
@@ -222,10 +218,10 @@
     </joint>
     <joint type="fixed" name="camera_joint">
-        <origin xyz="0.25 0 0" rpy="0 0 0"/>
+        <origin xyz="0.2 0 0" rpy="0 0 0"/>
         <child link="camera"/>
         <parent link="chassis"/>
     </joint>
     <joint type="fixed" name="hokuyo_joint">
-        <origin xyz="0.15 0 0.1" rpy="0 0 0"/>
+        <origin xyz="0.18 0 0.05" rpy="0 0 0"/>
         <child link="hokuyo"/>
         <parent link="chassis"/>

Commit message: updates

File: urdf/saminda_bot.xacro (robot description, xacro)
@@ -18,5 +18,5 @@
     </joint>
     <link name='chassis'>
-        <pose>0 0 0.1 0 0 0</pose>
+        <pose>0 0 0.025 0 0 0</pose>
         <inertial>
             <mass value="5.0"/>
@@ -186,5 +186,5 @@
     </link>
     <joint type="continuous" name="right_front">
-        <origin xyz="0.15 -0.13 0" rpy="0 0 0"/>
+        <origin xyz="0.10 -0.13 0" rpy="0 0 0"/>
         <child link="right_front_wheel"/>
         <parent link="chassis"/>
@@ -194,5 +194,5 @@
     </joint>
     <joint type="continuous" name="right_rear">
-        <origin xyz="-0.15 -0.13 0" rpy="0 0 0"/>
+        <origin xyz="-0.10 -0.13 0" rpy="0 0 0"/>
         <child link="right_rear_wheel"/>
         <parent link="chassis"/>
@@ -202,5 +202,5 @@
     </joint>
     <joint type="continuous" name="left_front">
-        <origin xyz="0.15 0.13 0" rpy="0 0 0"/>
+        <origin xyz="0.10 0.13 0" rpy="0 0 0"/>
         <child link="left_front_wheel"/>
         <parent link="chassis"/>
@@ -210,5 +210,5 @@
     </joint>
     <joint type="continuous" name="left_rear">
-        <origin xyz="-0.15 0.13 0" rpy="0 0 0"/>
+        <origin xyz="-0.10 0.13 0" rpy="0 0 0"/>
         <child link="left_rear_wheel"/>
         <parent link="chassis"/>

Commit message: update params

File: urdf/saminda_bot.xacro (robot description, xacro)
@@ -45,19 +45,19 @@
         <inertial>
             <mass value="0.2"/>
-             <origin xyz="0.0 0 0" rpy="1.5707 0 0"/>
-            <inertia
-                    ixx="0.005" ixy="0" ixz="0"
-                    iyy="0.005" iyz="0"
-                    izz="0.005"
-            />
-        </inertial>
-        <collision name='collision'>
-             <origin xyz="0 0 0" rpy="1.5707 0 0"/>
-            <geometry>
-                <cylinder length="0.0375" radius="0.055"/>
-            </geometry>
-        </collision>
-        <visual name='visual'>
-             <origin xyz="0 0 0" rpy="1.5707 0 0"/>
+             <origin xyz="0.0 0 0" rpy="0 1.5707 1.5707"/>
+            <inertia
+                    ixx="0.005" ixy="0" ixz="0"
+                    iyy="0.005" iyz="0"
+                    izz="0.005"
+            />
+        </inertial>
+        <collision name='collision'>
+             <origin xyz="0 0 0" rpy="0 1.5707 1.5707"/>
+            <geometry>
+                <cylinder length="0.0375" radius="0.055"/>
+            </geometry>
+        </collision>
+        <visual name='visual'>
+             <origin xyz="0 0 0" rpy="0 1.5707 1.5707"/>
             <geometry>
                 <cylinder length="0.0375" radius="0.055"/>
@@ -69,19 +69,19 @@
         <inertial>
             <mass value="0.2"/>
-             <origin xyz="0.0 0 0" rpy="1.5707 0 0"/>
-            <inertia
-                    ixx="0.005" ixy="0" ixz="0"
-                    iyy="0.005" iyz="0"
-                    izz="0.005"
-            />
-        </inertial>
-        <collision name='collision'>
-             <origin xyz="0 0 0" rpy="1.5707 0 0"/>
-            <geometry>
-                <cylinder length="0.0375" radius="0.055"/>
-            </geometry>
-        </collision>
-        <visual name='visual'>
-             <origin xyz="0 0 0" rpy="1.5707 0 0"/>
+             <origin xyz="0.0 0 0" rpy="0 1.5707 1.5707"/>
+            <inertia
+                    ixx="0.005" ixy="0" ixz="0"
+                    iyy="0.005" iyz="0"
+                    izz="0.005"
+            />
+        </inertial>
+        <collision name='collision'>
+             <origin xyz="0 0 0" rpy="0 1.5707 1.5707"/>
+            <geometry>
+                <cylinder length="0.0375" radius="0.055"/>
+            </geometry>
+        </collision>
+        <visual name='visual'>
+             <origin xyz="0 0 0" rpy="0 1.5707 1.5707"/>
             <geometry>
                 <cylinder length="0.0375" radius="0.055"/>
@@ -93,19 +93,19 @@
         <inertial>
             <mass value="0.2"/>
-             <origin xyz="0.0 0 0" rpy="1.5707 0 0"/>
-            <inertia
-                    ixx="0.005" ixy="0" ixz="0"
-                    iyy="0.005" iyz="0"
-                    izz="0.005"
-            />
-        </inertial>
-        <collision name='collision'>
-             <origin xyz="0 0 0" rpy="1.5707 0 0"/>
-            <geometry>
-                <cylinder length="0.0375" radius="0.055"/>
-            </geometry>
-        </collision>
-        <visual name='visual'>
-             <origin xyz="0 0 0" rpy="1.5707 0 0"/>
+             <origin xyz="0.0 0 0" rpy="0 1.5707 1.5707"/>
+            <inertia
+                    ixx="0.005" ixy="0" ixz="0"
+                    iyy="0.005" iyz="0"
+                    izz="0.005"
+            />
+        </inertial>
+        <collision name='collision'>
+             <origin xyz="0 0 0" rpy="0 1.5707 1.5707"/>
+            <geometry>
+                <cylinder length="0.0375" radius="0.055"/>
+            </geometry>
+        </collision>
+        <visual name='visual'>
+             <origin xyz="0 0 0" rpy="0 1.5707 1.5707"/>
             <geometry>
                 <cylinder length="0.0375" radius="0.055"/>
@@ -117,19 +117,19 @@
         <inertial>
             <mass value="0.2"/>
-             <origin xyz="0.0 0 0" rpy="1.5707 0 0"/>
-            <inertia
-                    ixx="0.005" ixy="0" ixz="0"
-                    iyy="0.005" iyz="0"
-                    izz="0.005"
-            />
-        </inertial>
-        <collision name='collision'>
-             <origin xyz="0 0 0" rpy="1.5707 0 0"/>
-            <geometry>
-                <cylinder length="0.0375" radius="0.055"/>
-            </geometry>
-        </collision>
-        <visual name='visual'>
-             <origin xyz="0 0 0" rpy="1.5707 0 0"/>
+             <origin xyz="0.0 0 0" rpy="0 1.5707 1.5707"/>
+            <inertia
+                    ixx="0.005" ixy="0" ixz="0"
+                    iyy="0.005" iyz="0"
+                    izz="0.005"
+            />
+        </inertial>
+        <collision name='collision'>
+             <origin xyz="0 0 0" rpy="0 1.5707 1.5707"/>
+            <geometry>
+                <cylinder length="0.0375" radius="0.055"/>
+            </geometry>
+        </collision>
+        <visual name='visual'>
+             <origin xyz="0 0 0" rpy="0 1.5707 1.5707"/>
             <geometry>
                 <cylinder length="0.0375" radius="0.055"/>
