Commit message: param update

File: urdf/saminda_bot.xacro (robot description, xacro)
@@ -1,152 +1,180 @@
-<?xml version='1.0'?>
-<robot name="saminda_bot" xmlns:xacro="http://www.ros.org/wiki/xacro">
+<?xml version="1.0"?>
+<robot xmlns:xacro="http://www.ros.org/wiki/xacro" name="saminda_bot">
+    <xacro:property name="base_mass" value="5"/> <!-- in kg-->
+    <xacro:property name="base_x_size" value="0.2"/>
+    <xacro:property name="base_y_size" value="0.3"/>
+    <xacro:property name="base_z_size" value="0.1"/>
+    <!-- Wheels -->
+    <xacro:property name="wheel_mass" value="1"/> <!-- in kg-->
+    <xacro:property name="length_wheel" value="0.05"/>
+    <xacro:property name="radius_wheel" value="0.05"/>
+    <xacro:property name="camera_link" value="0.05"/>
+    <xacro:macro name="default_inertial" params="mass">
+        <inertial>
+            <mass value="${mass}"/>
+            <inertia ixx="1.0" ixy="0.0" ixz="0.0"
+                     iyy="1.0" iyz="0.0"
+                     izz="1.0"/>
+        </inertial>
+    </xacro:macro>
+    <macro name="box_inertia" params="m x y z">
+        <inertia ixx="${m*(y*y+z*z)/12}" ixy="0" ixz="0"
+                 iyy="${m*(x*x+z*z)/12}" iyz="0"
+                 izz="${m*(x*x+z*z)/12}"/>
+    </macro>
+    <macro name="cylinder_inertia" params="m r h">
+        <inertia ixx="${m*(3*r*r+h*h)/12}" ixy="0" ixz="0"
+                 iyy="${m*(3*r*r+h*h)/12}" iyz="0"
+                 izz="${m*r*r/2}"/>
+    </macro>
+    <link name="robot_footprint">
+        <visual>
+            <geometry>
+                <box size="0.001 0.001 0.001"/>
+            </geometry>
+            <origin rpy="0 0 0" xyz="0 0 0"/>
+        </visual>
+    </link>
     <xacro:include filename="$(find udacity_bot)/urdf/saminda_bot.gazebo"/>
-    <material name="red">
-        <color rgba="1 0 0 1"/>
-    </material>
-    <material name="green">
-        <color rgba="0 1 0 1"/>
-    </material>
-    <material name="blue">
-        <color rgba="0 0 1 1"/>
-    </material>
-    <link name="robot_footprint"></link>
     <joint name="robot_footprint_joint" type="fixed">
-        <origin xyz="0 0 0" rpy="0 0 0"/>
+        <origin xyz="0 0 0.15"/>
         <parent link="robot_footprint"/>
         <child link="chassis"/>
     </joint>
-    <link name='chassis'>
-        <pose>0 0 0.025 0 0 0</pose>
-        <inertial>
-            <mass value="5.0"/>
-            <origin xyz="0.0 0 0" rpy=" 0 0 0"/>
-            <inertia
-                    ixx="0.1" ixy="0" ixz="0"
-                    iyy="0.1" iyz="0"
-                    izz="0.1"
-            />
-        </inertial>
-        <collision name='collision'>
-            <origin xyz="0 0 0" rpy=" 0 0 0"/>
-            <geometry>
-                <box size="0.4 0.2 0.05"/>
-            </geometry>
-        </collision>
-        <visual name='visual'>
-            <origin xyz="0 0 0" rpy=" 0 0 0"/>
-            <geometry>
-                <box size="0.4 0.2 0.05"/>
-            </geometry>
-            <material name="blue"/>
-        </visual>
-    </link>
-    <link name='right_front_wheel'>
-        <inertial>
-            <mass value="0.2"/>
-             <origin xyz="0.0 0 0" rpy="0 1.5707 1.5707"/>
-            <inertia
-                    ixx="0.005" ixy="0" ixz="0"
-                    iyy="0.005" iyz="0"
-                    izz="0.005"
-            />
-        </inertial>
-        <collision name='collision'>
-             <origin xyz="0 0 0" rpy="0 1.5707 1.5707"/>
-            <geometry>
-                <cylinder length="0.0375" radius="0.055"/>
-            </geometry>
-        </collision>
-        <visual name='visual'>
-             <origin xyz="0 0 0" rpy="0 1.5707 1.5707"/>
-            <geometry>
-                <cylinder length="0.0375" radius="0.055"/>
-            </geometry>
-            <material name="green"/>
-        </visual>
-    </link>
-    <link name='left_front_wheel'>
-        <inertial>
-            <mass value="0.2"/>
-             <origin xyz="0.0 0 0" rpy="0 1.5707 1.5707"/>
-            <inertia
-                    ixx="0.005" ixy="0" ixz="0"
-                    iyy="0.005" iyz="0"
-                    izz="0.005"
-            />
-        </inertial>
-        <collision name='collision'>
-             <origin xyz="0 0 0" rpy="0 1.5707 1.5707"/>
-            <geometry>
-                <cylinder length="0.0375" radius="0.055"/>
-            </geometry>
-        </collision>
-        <visual name='visual'>
-             <origin xyz="0 0 0" rpy="0 1.5707 1.5707"/>
-            <geometry>
-                <cylinder length="0.0375" radius="0.055"/>
-            </geometry>
-            <material name="green"/>
-        </visual>
-    </link>
-    <link name='right_rear_wheel'>
-        <inertial>
-            <mass value="0.2"/>
-             <origin xyz="0.0 0 0" rpy="0 1.5707 1.5707"/>
-            <inertia
-                    ixx="0.005" ixy="0" ixz="0"
-                    iyy="0.005" iyz="0"
-                    izz="0.005"
-            />
-        </inertial>
-        <collision name='collision'>
-             <origin xyz="0 0 0" rpy="0 1.5707 1.5707"/>
-            <geometry>
-                <cylinder length="0.0375" radius="0.055"/>
-            </geometry>
-        </collision>
-        <visual name='visual'>
-             <origin xyz="0 0 0" rpy="0 1.5707 1.5707"/>
-            <geometry>
-                <cylinder length="0.0375" radius="0.055"/>
-            </geometry>
-            <material name="green"/>
-        </visual>
-    </link>
-    <link name='left_rear_wheel'>
-        <inertial>
-            <mass value="0.2"/>
-             <origin xyz="0.0 0 0" rpy="0 1.5707 1.5707"/>
-            <inertia
-                    ixx="0.005" ixy="0" ixz="0"
-                    iyy="0.005" iyz="0"
-                    izz="0.005"
-            />
-        </inertial>
-        <collision name='collision'>
-             <origin xyz="0 0 0" rpy="0 1.5707 1.5707"/>
-            <geometry>
-                <cylinder length="0.0375" radius="0.055"/>
-            </geometry>
-        </collision>
-        <visual name='visual'>
-             <origin xyz="0 0 0" rpy="0 1.5707 1.5707"/>
-            <geometry>
-                <cylinder length="0.0375" radius="0.055"/>
-            </geometry>
-            <material name="green"/>
-        </visual>
-    </link>
-    <link name='camera'>
-        <inertial>
-            <mass value="0.1"/>
-            <origin xyz="0.0 0 0" rpy="0 0 0"/>
-            <inertia
-                    ixx="1e-6" ixy="0" ixz="0"
-                    iyy="1e-6" iyz="0"
-                    izz="1e-6"
-            />
-        </inertial>
-        <collision name='camera_collision'>
+    <link name="chassis">
+        <visual>
+            <geometry>
+                <box size="${base_x_size} ${base_y_size} ${base_z_size}"/>
+            </geometry>
+            <origin rpy="0 0 1.54" xyz="0 0 0.05"/>
+            <material name="blue">
+                <color rgba="0 0 1 1"/>
+            </material>
+        </visual>
+        <collision>
+            <geometry>
+                <box size="${base_x_size} ${base_y_size} ${base_z_size}"/>
+            </geometry>
+        </collision>
+        <inertial>
+            <mass value="${base_mass}"/>
+            <origin xyz="0 0 0"/>
+            <!--The 3x3 rotational inertia matrix. -->
+            <box_inertia m="${base_mass}" x="${base_x_size}" y="${base_y_size}" z="${base_z_size}"/>
+        </inertial>
+    </link>
+    <link name="left_front_wheel">
+        <visual>
+            <geometry>
+                <cylinder length="${length_wheel}" radius="${radius_wheel}"/>
+            </geometry>
+            <origin rpy="0 0 0" xyz="0 0 0"/>
+            <material name="black">
+                <color rgba="0 0 0 1"/>
+            </material>
+        </visual>
+        <collision>
+            <geometry>
+                <cylinder length="${length_wheel}" radius="${radius_wheel}"/>
+            </geometry>
+        </collision>
+        <inertial>
+            <mass value="${wheel_mass}"/>
+            <origin xyz="0 0 0"/>
+            <cylinder_inertia m="${wheel_mass}" r="${radius_wheel}" h="${length_wheel}"/>
+        </inertial>
+    </link>
+    <link name="left_rear_wheel">
+        <visual>
+            <geometry>
+                <cylinder length="${length_wheel}" radius="${radius_wheel}"/>
+            </geometry>
+            <origin rpy="0 0 0" xyz="0 0 0"/>
+            <material name="black"/>
+        </visual>
+        <collision>
+            <geometry>
+                <cylinder length="${length_wheel}" radius="${radius_wheel}"/>
+            </geometry>
+        </collision>
+        <inertial>
+            <mass value="${wheel_mass}"/>
+            <origin xyz="0 0 0"/>
+            <cylinder_inertia m="${wheel_mass}" r="${radius_wheel}" h="${length_wheel}"/>
+        </inertial>
+    </link>
+    <link name="right_front_wheel">
+        <visual>
+            <geometry>
+                <cylinder length="${length_wheel}" radius="${radius_wheel}"/>
+            </geometry>
+            <origin rpy="0 0 0" xyz="0 0 0"/>
+            <material name="black"/>
+        </visual>
+        <collision>
+            <geometry>
+                <cylinder length="${length_wheel}" radius="${radius_wheel}"/>
+            </geometry>
+        </collision>
+        <inertial>
+            <mass value="${wheel_mass}"/>
+            <origin xyz="0 0 0"/>
+            <cylinder_inertia m="${wheel_mass}" r="${radius_wheel}" h="${length_wheel}"/>
+        </inertial>
+    </link>
+    <link name="right_rear_wheel">
+        <visual>
+            <geometry>
+                <cylinder length="${length_wheel}" radius="${radius_wheel}"/>
+            </geometry>
+            <origin rpy="0 0 0" xyz="0 0 0"/>
+            <material name="black"/>
+        </visual>
+        <collision>
+            <geometry>
+                <cylinder length="${length_wheel}" radius="${radius_wheel}"/>
+            </geometry>
+        </collision>
+        <inertial>
+            <mass value="${wheel_mass}"/>
+            <origin xyz="0 0 0"/>
+            <cylinder_inertia m="${wheel_mass}" r="${radius_wheel}" h="${length_wheel}"/>
+        </inertial>
+    </link>
+    <joint name="left_front" type="continuous">
+        <parent link="chassis"/>
+        <child link="left_front_wheel"/>
+        <origin rpy="-1.5707 0 0" xyz="0.1 0.13 0"/>
+        <axis xyz="0 0 1"/>
+    </joint>
+    <joint name="left_rear" type="continuous">
+        <axis xyz="0 0 1"/>
+        <anchor xyz="0 0 0"/>
+        <limit effort="100" velocity="100"/>
+        <parent link="chassis"/>
+        <child link="left_rear_wheel"/>
+        <origin rpy="-1.5707 0 0" xyz="-0.1 0.13 0"/>
+    </joint>
+    <joint name="right_front" type="continuous">
+        <parent link="chassis"/>
+        <axis xyz="0 0 1"/>
+        <child link="right_front_wheel"/>
+        <origin rpy="-1.5707 0 0" xyz="0.1 -0.13 0"/>
+    </joint>
+    <joint name="right_rear" type="continuous">
+        <parent link="chassis"/>
+        <axis xyz="0 0 1"/>
+        <child link="right_rear_wheel"/>
+        <origin rpy="-1.5707 0 0" xyz="-0.1 -0.13 0"/>
+    </joint>
+    <!-- Camera joint -->
+    <joint name="camera_joint" type="fixed">
+        <origin xyz="0.125 0 0.125" rpy="0 0 0"/>
+        <parent link="chassis"/>
+        <child link="camera"/>
+    </joint>
+    <!-- Camera -->
+    <link name="camera">
+        <collision>
             <origin xyz="0 0 0" rpy="0 0 0"/>
             <geometry>
@@ -154,76 +182,44 @@
             </geometry>
         </collision>
-        <visual name='camera_visual'>
+        <visual>
             <origin xyz="0 0 0" rpy="0 0 0"/>
             <geometry>
                 <box size="0.05 0.05 0.05"/>
             </geometry>
-            <material name="red"/>
-        </visual>
-    </link>
-    <link name='hokuyo'>
-        <inertial>
-            <mass value="0.1"/>
-            <origin xyz="0.0 0 0" rpy="0 0 0"/>
-            <inertia
-                    ixx="1e-6" ixy="0" ixz="0"
-                    iyy="1e-6" iyz="0"
-                    izz="1e-6"
-            />
-        </inertial>
-        <collision name='hokuyo_collision'>
-            <origin xyz="0 0 0" rpy="0 0 0"/>
-            <geometry>
-                <box size="0.1 0.1 0.1"/>
-            </geometry>
-        </collision>
-        <visual name='hokuyo_visual'>
-            <origin xyz="0 0 0" rpy="0 0 0"/>
+            <material name="red">
+                <color rgba="1 0 0 1"/>
+            </material>
+        </visual>
+        <inertial>
+            <mass value="1e-5"/>
+            <origin xyz="0 0 0" rpy="0 0 0"/>
+            <inertia ixx="1e-6" ixy="0" ixz="0" iyy="1e-6" iyz="0" izz="1e-6"/>
+        </inertial>
+    </link>
+    <!-- Hokuyo joint -->
+    <joint name="hokuyo_joint" type="fixed">
+        <origin xyz="0.125 0.05 0.125" rpy="0 0 0"/>
+        <parent link="chassis"/>
+        <child link="hokuyo"/>
+    </joint>
+    <!-- Hokuyo Laser -->
+    <link name="hokuyo">
+        <collision>
+            <origin xyz="0 0 0" rpy="0 0 0"/>
+            <geometry>
+                <box size="0.0 -0.05 0.06"/>
+            </geometry>
+        </collision>
+        <visual>
+            <origin xyz="0 -0.05 0.06" rpy="0 0 0"/>
             <geometry>
                 <mesh filename="package://udacity_bot/meshes/hokuyo.dae"/>
             </geometry>
         </visual>
-    </link>
-    <joint type="continuous" name="right_front">
-        <origin xyz="0.10 -0.13 0" rpy="0 0 0"/>
-        <child link="right_front_wheel"/>
-        <parent link="chassis"/>
-        <axis xyz="0 1 0" rpy="0 0 0" use_parent_model_frame="true"/>
-        <limit effort="10000" velocity="1000"/>
-        <dynamics damping="1.0" friction="1.0"/>
-    </joint>
-    <joint type="continuous" name="right_rear">
-        <origin xyz="-0.10 -0.13 0" rpy="0 0 0"/>
-        <child link="right_rear_wheel"/>
-        <parent link="chassis"/>
-        <axis xyz="0 1 0" rpy="0 0 0" use_parent_model_frame="true"/>
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